File: GridTiedBatteryBoostConverter.kicad_pcb (KiCad board)
At the start: 2 copper layers, 270.1 x 143.1 mm, 116 parts, among them J101 Battery Connection, J103 Solar Panels, J401 Screw_Terminal_01x02, J402 AudioJack2_SwitchT, Q101 IXFP36N20X3, Q102 BC847B-13-F, Q103 SSM3K329R, Q104 SSM3J334R, Q201 SSM3K329R, Q202 SSM3K329R, Q203 SSM3J334R, Q301 BC847B-13-F, Q302 BC856B-13-F, Q305 TK32A12N1,S4X, Q306 TK32A12N1,S4X, SW201 SW_Push, SW202 SW_Push, SW203 SW_Push, U101 OPA2837DGK, U102 UCC2800DTR, U201 LCD 2004A, U202 Teensy-LC, U203 wizfi360, U301 FDA217, U302 LTC7138EMSE-PBF, U303 TPS560200, U304 TLV70430_SOT23-5

Commit message: started routing backing up tonnes of changes,2.048V reference changed to 2.5V ref, to match ucc2800, cos to change to a version with a 2V feedback, would require me to update the Oscillator cap and resistor,and also recalulate the class 2 loop compensation components etc.  Move the location of the teensy LC and added the ESP-WROOM-o2 wifi module.
Parts:
- removed R403: 1K ohms .1%, Resistors_SMD:R_0805_HandSoldering
- added C201: 1uF x7r 16V, Capacitors_SMD:C_0805_HandSoldering, F.Cu at (131.2, 203.1)
- added C202: 0.1uF x7r 16V, Capacitors_SMD:C_0805_HandSoldering, F.Cu at (131.2, 207.9)
- added C203: 0.1uF x7r 16V, Capacitors_SMD:C_0805_HandSoldering, F.Cu at (43.6, 136.3)
- added C204: 10uF 16V X7R, Capacitors_SMD:C_1206_HandSoldering, F.Cu at (40.0, 143.2)
- added C205: 0.1uF x7r 16V, Capacitors_SMD:C_0805_HandSoldering, F.Cu at (27.0, 116.2)
- added C301: 10uF 16V X7R, Capacitors_SMD:C_1206_HandSoldering, F.Cu at (92.4, 103.0)
- added C302: 0.47uF x7r 25V 10%, Capacitors_SMD:C_0805_HandSoldering, F.Cu at (166.6, 96.9)
- added C304: 0.1uF 16V X7R, Capacitors_SMD:C_0805_HandSoldering, F.Cu at (89.8, 103.4)
- added C305: 10uF X7R 16V, Capacitors_SMD:C_1206_HandSoldering, F.Cu at (78.1, 109.0)
- added C307: 10uF X7R 16V, Capacitors_SMD:C_1206_HandSoldering, F.Cu at (75.6, 108.9)
- added J202: Conn_01x03_Female, Pin_Headers:Pin_Header_Straight_1x03_Pitch2.54mm, F.Cu at (43.3, 121.7)
- added J203: I2C_BUS, Pin_Headers:Pin_Header_Straight_1x04_Pitch2.54mm, F.Cu at (153.3, 101.0)
- added JP201: SDA_EN, Pin_Headers:Pin_Header_Straight_1x02_Pitch2.54mm, F.Cu at (29.2, 180.0)
- added JP202: SCL_EN, Pin_Headers:Pin_Header_Straight_1x02_Pitch2.54mm, F.Cu at (33.8, 180.0)
- added JP203: BOOT_OPTION, Pin_Headers:Pin_Header_Straight_1x02_Pitch2.54mm, F.Cu at (24.5, 180.0)
- added L303: 15uH 730mA Sat, Inductors_jl:Inductor_1210_HandSoldering, F.Cu at (82.9, 107.1)
- added R208: 4k7 1%, Resistors_SMD:R_0805_HandSoldering, F.Cu at (52.1, 183.4)
- added R209: 15K 1%, Resistors_SMD:R_0805_HandSoldering, F.Cu at (39.0, 179.1)
- added R210: 15K 1%, Resistors_SMD:R_0805_HandSoldering, F.Cu at (47.9, 140.9)
- added R211: 4k7 1%, Resistors_SMD:R_0805_HandSoldering, F.Cu at (160.9, 95.6)
- added R212: 4k7 1%, Resistors_SMD:R_0805_HandSoldering, F.Cu at (157.3, 95.6)
- added R213: 15K 1%, Resistors_SMD:R_0805_HandSoldering, F.Cu at (26.9, 110.7)
- added R303: 61.9k 0.1%, Resistors_SMD:R_0805_HandSoldering, F.Cu at (77.0, 102.0)
- added R304: 20k 0.1%, Resistors_SMD:R_0805_HandSoldering, F.Cu at (81.6, 103.0)
- added U204: ESP-WROOM-02, RF_Module:ESP-WROOM-02, F.Cu at (31.2, 150.6)
- added U305: REF2925AIDBZT, Package_TO_SOT_SMD:SOT-23_Handsoldering, F.Cu at (166.3, 101.0)
- added U306: TPS560200, Package_TO_SOT_SMD:SOT-23-5_HandSoldering, F.Cu at (86.2, 103.6)
- L302: value 15uH 600mA Sat -> 15uH 730mA Sat
- R401: value 10K ohms .1% -> 5.9K ohms .1%
- R404: value 47 Ohms 0.1% -> 41.2 Ohms 0.1%
- SW201: value SW_Push -> SW_Up
- SW202: value SW_Push -> SW_Down
- SW203: value SW_Push -> SW_Enter
- U203: value wizfi360 -> PCF8574ADWR; footprint WIZnet:wiznet360-pa -> Housings_SOIC:SOIC-16W_7.5x10.3mm_Pitch1.27mm
- moved SW203 156.4 mm to (194.1, 154.8)
- moved SW201 125.3 mm to (52.5, 154.7)
- moved U203 102.7 mm to (123.7, 127.0), turned to 0 degrees
- moved U202 39.5 mm to (165.6, 113.6), turned to 0 degrees
- moved D401 34.2 mm to (187.2, 117.5)
- moved D402 26.6 mm to (193.4, 114.7)
- moved Q203 22.9 mm to (146.1, 139.4)
- moved R207 22.9 mm to (151.9, 140.9)
- moved Q201 22.9 mm to (151.6, 136.1)
- moved R205 22.9 mm to (146.2, 135.7)
- moved R201 15.9 mm to (123.2, 140.8)
- moved R206 15.9 mm to (113.0, 140.8)
- moved RV201 15.9 mm to (168.4, 140.9)
- moved U201 15.9 mm to (148.6, 146.6)
- moved Q202 15.9 mm to (108.6, 140.6)
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Connections:
- net /Sheet5F4EB1AB/Vout renamed /Vout
- net /Sheet5F4EB1AB/Vsolar_in renamed /Vsolar_in
- J402 pad RN: Net-(C401-Pad1) -> (no net)
- J402 pad TN: Net-(C401-Pad1) -> (no net)
- R206 pad 1: Net-(R206-Pad1) -> Net-(Q202-Pad3)
- R402 pad 2: Net-(R402-Pad2) -> Net-(C401-Pad1)
- R405 pad 1: +3.3V_TEENSY_OUT -> /+2.5V_REF
- U201 pad 15: Net-(R206-Pad1) -> Net-(U201-Pad15)
- U201 pad 4: /Teensy-LC/LCD_RS -> Net-(U201-Pad4)
- U201 pad 5: /Teensy-LC/LCD_RW -> Net-(U201-Pad5)
- U201 pad 6: /Teensy-LC/LCD_EN -> Net-(U201-Pad6)
- U202 pad 12: Net-(U202-Pad12) -> Net-(SW201-Pad2)
- U202 pad 2: Net-(U202-Pad2) -> Net-(J202-Pad1)
- U202 pad 23: LCD_ON_OFF -> Mains_Voltage
- U202 pad 24: /Teensy-LC/LCD_DB7 -> Mains_Current
- U202 pad 25: /Teensy-LC/LCD_DB6 -> Net-(U202-Pad25)
- U202 pad 26: /Teensy-LC/LCD_DB5 -> Net-(U202-Pad26)
- U202 pad 27: /Teensy-LC/LCD_EN -> /Teensy-LC/BOOST_ON_OFF
- U202 pad 28: /Teensy-LC/LCD_RW -> Net-(U202-Pad28)
- U202 pad 29: Net-(U202-Pad29) -> SCL1
- U202 pad 3: Net-(U202-Pad3) -> Net-(J202-Pad2)
- U202 pad 30: Net-(SW201-Pad2) -> SDA1
- U202 pad 35: Net-(U202-Pad35) -> /+2.5V_REF
- U202 pad 36: Mains_Current -> Net-(U202-Pad36)
- U202 pad 37: Mains_Voltage -> Net-(U202-Pad37)
- U202 pad 6: /Teensy-LC/LCD_RS -> Net-(U202-Pad6)
- U202 pad 7: /Teensy-LC/BOOST_ON_OFF -> Net-(U202-Pad7)
- U202 pad 8: /Teensy-LC/LCD_DB4 -> Net-(U202-Pad8)
- U203 pad 1: Net-(U203-Pad1) -> 0
- U203 pad 10: Net-(U203-Pad10) -> /Teensy-LC/LCD_RW
- U203 pad 11: Net-(U203-Pad11) -> /Teensy-LC/LCD_RS
- U203 pad 12: Net-(U203-Pad12) -> LCD_ON_OFF
- U203 pad 14: Net-(U203-Pad14) -> SCL1
- U203 pad 15: Net-(U203-Pad15) -> SDA1
- U203 pad 16: Net-(U203-Pad16) -> +3.3V_TEENSY_OUT
- U203 pad 2: Net-(U203-Pad2) -> 0
- U203 pad 3: Net-(U203-Pad3) -> 0
- U203 pad 4: Net-(U203-Pad4) -> /Teensy-LC/LCD_DB4
- U203 pad 5: Net-(U203-Pad5) -> /Teensy-LC/LCD_DB5
- U203 pad 6: Net-(U203-Pad6) -> /Teensy-LC/LCD_DB6
- U203 pad 7: Net-(U203-Pad7) -> /Teensy-LC/LCD_DB7
- U203 pad 8: Net-(U203-Pad8) -> 0
- U203 pad 9: Net-(U203-Pad9) -> /Teensy-LC/LCD_EN
Routing:
- net Net-(SW203-Pad1): track 189.9 -> 42.3 mm, vias 6 -> 2
- net LCD_ON_OFF: track 153.4 -> 16.1 mm, vias 4 -> 2
- net Net-(SW201-Pad2): track 16.0 -> 147.4 mm
- net /PowerSupplies/CHARGER_ON_OFF: track 171.8 -> 66.7 mm
- net /+2.5V_REF: track 0.00 -> 98.0 mm, vias 0 -> 2
- net +5V: track 333.4 -> 240.8 mm, vias 2 -> 0
- net Mains_Current: track 72.4 -> 125.0 mm, vias 2 -> 0
- net Net-(SW201-Pad1): track 51.4 -> 0.00 mm, vias 2 -> 0
- net Mains_Voltage: track 21.7 -> 63.9 mm
- net /Teensy-LC/BOOST_ON_OFF: track 75.2 -> 40.7 mm, vias 4 -> 2
- net Net-(SW202-Pad1): track 60.1 -> 35.1 mm, vias 4 -> 0
- net SCL1: track 0.00 -> 24.7 mm, vias 0 -> 1
- net SDA1: track 0.00 -> 21.3 mm
- net +3.3V_TEENSY_OUT: track 37.2 -> 18.8 mm
- net Net-(Q203-Pad3): track 27.0 -> 10.2 mm, vias 2 -> 0
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- added copper zone on B.Cu, net SCL1
- removed copper zone on B.Cu, net 0
Other:
- outline, holes or cut-outs redrawn

Commit message: Almost finished the routing, an other backup commit git add *
Parts:
- U204: value ESP-WROOM-02 -> ESP-WROOM-02U; footprint RF_Module:ESP-WROOM-02 -> RF_Module_jl:MODULE_ESP-WROOM-02U
- moved R208 105.0 mm to (139.9, 125.8), turned to 180 degrees
- moved C202 80.8 mm to (142.8, 128.0)
- moved C201 74.1 mm to (142.8, 129.9)
- moved R303 52.6 mm to (24.4, 103.9)
- moved C301 52.6 mm to (39.9, 105.2)
- moved L303 52.6 mm to (30.4, 109.3)
- moved C304 52.6 mm to (37.3, 105.7)
- moved C305 52.6 mm to (25.6, 111.2)
- moved C307 52.6 mm to (23.1, 111.2)
- moved R304 52.6 mm to (29.1, 105.2)
- moved U306 52.6 mm to (33.7, 105.8)
- moved R209 46.9 mm to (40.2, 132.2)
- moved JP202 46.7 mm to (29.8, 133.5), turned to 90 degrees
- moved JP203 43.5 mm to (38.1, 138.7), turned to 180 degrees
- moved JP201 42.4 mm to (29.8, 137.6), turned to 90 degrees
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Connections:
- net Net-(C203-Pad1) renamed /Teensy-LC/wifi_en
- net Net-(C205-Pad1) renamed /Teensy-LC/~reset
- net Net-(J202-Pad1) renamed /Teensy-LC/mcu_wifi_rx
- net Net-(J202-Pad2) renamed /Teensy-LC/mcu_wifi_tx
- R206 pad 1: Net-(Q202-Pad3) -> Net-(R206-Pad1)
- U201 pad 15: Net-(U201-Pad15) -> Net-(R206-Pad1)
- U201 pad 4: Net-(U201-Pad4) -> /Teensy-LC/LCD_RS
- U201 pad 5: Net-(U201-Pad5) -> /Teensy-LC/LCD_RW
- U201 pad 6: Net-(U201-Pad6) -> /Teensy-LC/LCD_EN
Routing:
- net SDA1: track 21.3 -> 216.4 mm, vias 0 -> 2
- net SCL1: track 24.7 -> 209.1 mm, vias 1 -> 6
- net +5V: track 240.8 -> 414.9 mm, vias 0 -> 2
- net /Teensy-LC/wifi_en: track 0.00 -> 145.8 mm, vias 0 -> 2
- net +11V: track 60.3 -> 177.4 mm
- net /Teensy-LC/mcu_wifi_tx: track 0.00 -> 100.1 mm
- net /Teensy-LC/mcu_wifi_rx: track 0.00 -> 99.5 mm
- net +3.3V_wifi_only: track 0.00 -> 68.9 mm
- net /PowerSupplies/CHARGER_ON_OFF: track 66.7 -> 0.00 mm, vias 4 -> 0
- net +3.3V_TEENSY_OUT: track 18.8 -> 66.1 mm, vias 0 -> 1
- net 0: track 214.6 -> 253.7 mm, vias 60 -> 80
- net LCD_ON_OFF: track 16.1 -> 50.7 mm, vias 2 -> 0
- net /Teensy-LC/LCD_DB4: track 0.00 -> 23.7 mm
- net /Teensy-LC/LCD_DB5: track 0.00 -> 21.9 mm
- net Net-(C314-Pad2): track 74.6 -> 93.5 mm, vias 1 -> 4
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- added copper zone on B.Cu, net 0
- removed copper zone on B.Cu, net SCL1
Other:
- board text added: "Gnd"
- board text added: "Rx"
- board text added: "Tx"

Commit message: Finish routing finally
Parts:
- moved C305 2.55 mm to (25.7, 108.7), turned to 90 degrees
- moved C307 2.55 mm to (23.1, 108.6), turned to 90 degrees
Routing:
- net /PowerSupplies/CHARGER_ON_OFF: track 0.00 -> 115.4 mm, vias 0 -> 4
- net Net-(R303-Pad2): track 3.32 -> 10.3 mm
- net 0: track 253.7 -> 260.2 mm, vias 80 -> 90
- net +3.3V_wifi_only: track 68.9 -> 73.4 mm
- net SCL1: track 209.1 -> 211.5 mm
- net +3.3V_TEENSY_OUT: track 66.1 -> 64.4 mm, vias 1 -> 3
- net SDA1: track 216.4 -> 216.7 mm, vias 2 -> 4

Commit message: fixed a few DRC errors, introduced error by adding edge.cuts to the buttons footprint, now warns board outline not complete.  3d wont completely render also because of this.
Parts:
- J103: value Solar Panels -> + Solar Panels -
- moved R201 0.50 mm to (124.5, 143.8)
- moved Ct101 0.15 mm to (189.6, 69.7)
Routing:
- net +3.3V_TEENSY_OUT: track 64.4 -> 67.5 mm
Other:
- board text added: "- Inverter +"
- board text added: "I2C_BUS 3.3V GND SDA1 SCL"
- board text removed: "Inverter"

Commit message: added mounting holes, should have done that sort of thing right at start.
Parts:
- added REF**: MountingHole_3.2mm_M3_Pad, Mounting_Holes:MountingHole_3.2mm_M3_Pad, F.Cu at (141.8, 91.8)
- added REF**: MountingHole_3.2mm_M3_Pad, Mounting_Holes:MountingHole_3.2mm_M3_Pad, F.Cu at (278.1, 19.5)
- added REF**: MountingHole_3.2mm_M3_Pad, Mounting_Holes:MountingHole_3.2mm_M3_Pad, F.Cu at (278.1, 152.6)
- added REF**: MountingHole_3.2mm_M3_Pad, Mounting_Holes:MountingHole_3.2mm_M3_Pad, F.Cu at (18.0, 19.5)
- added REF**: MountingHole_3.2mm_M3_Pad, Mounting_Holes:MountingHole_3.2mm_M3_Pad, F.Cu at (18.0, 152.5)
- moved J101 8.56 mm to (19.4, 30.1)
- moved J401 7.26 mm to (272.5, 122.9)
- moved C104 6.75 mm to (255.2, 27.1)
- moved J402 6.69 mm to (276.9, 140.4)
- moved REF*** 5.08 mm to (267.6, 152.6)
Routing:
- net Vboost_out: track 158.8 -> 175.7 mm
- net Vin: track 251.4 -> 240.1 mm
- net ChargerConnection: track 43.9 -> 35.2 mm
- net Net-(C401-Pad1): track 106.0 -> 114.4 mm
- net Net-(J401-Pad1): track 15.9 -> 24.3 mm
- net Mains_Current: track 125.0 -> 130.4 mm
- net Net-(J401-Pad2): track 12.8 -> 13.8 mm

Commit message: added testpoints
Parts:
- added TP101: TestPoint, Measurement_Points:Measurement_Point_Square-SMD-Pad_Big, F.Cu at (194.7, 102.7)
- added TP102: TestPoint, Measurement_Points:Measurement_Point_Square-SMD-Pad_Big, F.Cu at (194.8, 72.5)
- added TP103: TestPoint, Measurement_Points:Measurement_Point_Square-SMD-Pad_Big, F.Cu at (184.6, 98.2)
- added TP201: TestPoint, Measurement_Points:Measurement_Point_Square-SMD-Pad_Big, F.Cu at (118.3, 128.2)
- added TP202: TestPoint, Measurement_Points:Measurement_Point_Square-SMD-Pad_Big, F.Cu at (153.9, 126.0)
- added TP203: TestPoint, Measurement_Points:Measurement_Point_Square-SMD-Pad_Big, F.Cu at (171.8, 100.7)
- added TP301: TestPoint, Measurement_Points:Measurement_Point_Square-SMD-Pad_Big, F.Cu at (37.2, 99.9)
- added TP302: TestPoint, Measurement_Points:Measurement_Point_Square-SMD-Pad_Big, F.Cu at (28.8, 113.0)
- added TP303: TestPoint, Measurement_Points:Measurement_Point_Square-SMD-Pad_Big, F.Cu at (110.7, 90.9)
- added TP304: TestPoint, Measurement_Points:Measurement_Point_Square-SMD-Pad_Big, F.Cu at (148.3, 68.7)
- added TP305: TestPoint, Measurement_Points:Measurement_Point_Square-SMD-Pad_Big, F.Cu at (185.1, 124.9)
- added TP306: TestPoint, Measurement_Points:Measurement_Point_Square-SMD-Pad_Big, F.Cu at (86.2, 93.8)
- added TP307: TestPoint, Measurement_Points:Measurement_Point_Square-SMD-Pad_Big, F.Cu at (167.8, 87.2)
- J103: value + Solar Panels - -> Solar Panels
Connections:
- C104 pad 2: 0 -> Net-(C104-Pad3)
Routing:
- net Net-(R308-Pad2): track 7.31 -> 23.8 mm
- net Net-(R303-Pad2): track 10.3 -> 15.2 mm
