File: SolarDCSwitch.sch (KiCad schematic (older format))
At the start: 3 parts

Commit message: Consolidated a lot of part values that were the same part but not detected the same by Boms_away BOM editor because of subtle differences in how I specified the values. Added Digi-key part numbers to the resistors. Replaced 2mOhm .5W current sense resistors with 1W 2mOhm Thin Film resistors (lower inductance than metal element), And fixed a bug where I was earthing the return feed of the Solar inverter before passing through the current sense resistor.
Parts:
- D501, D502, D503: MFR (none) -> -; MPN (none) -> -; SPN (none) -> -; SPR (none) -> -; SPURL (none) -> -
Changed lines of the file:
@@
 Comment4 ""
 $EndDescr
-Text Notes 6700 3750 2    50   ~ 0
-Solar 585V 8A Max
-Text HLabel 2750 3900 0    50   Input ~ 0
-Vbattery_in
-Text HLabel 6000 3900 2    50   Input ~ 0
-Vsolar_in
-Text HLabel 4350 2900 1    50   Output ~ 0
-Vout
 $Comp
 L Device:D_Schottky D?
@@
 F 2 "Diodes_ThroughHole_jl:Diode_TO_220AC_Horizonal" H 3250 3900 50  0001 C CNN
 F 3 "http://www.vishay.com/docs/96244/vs-20etsm3_vs-20atsm3.pdf" H 3250 3900 50  0001 C CNN
+F 4 "-" H 0   0   50  0001 C CNN "MFR"
+F 5 "-" H 0   0   50  0001 C CNN "MPN"
+F 6 "-" H 0   0   50  0001 C CNN "SPR"
+F 7 "-" H 0   0   50  0001 C CNN "SPN"
+F 8 "-" H 0   0   50  0001 C CNN "SPURL"
 	1    3250 3900
 	-1   0    0    1
@@
 F 2 "Diodes_ThroughHole_jl:Diode_TO_220AC_Horizonal" H 5250 3900 50  0001 C CNN
 F 3 "http://www.vishay.com/docs/96244/vs-20etsm3_vs-20atsm3.pdf" H 5250 3900 50  0001 C CNN
+F 4 "-" H 0   0   50  0001 C CNN "MFR"
+F 5 "-" H 0   0   50  0001 C CNN "MPN"
+F 6 "-" H 0   0   50  0001 C CNN "SPR"
+F 7 "-" H 0   0   50  0001 C CNN "SPN"
+F 8 "-" H 0   0   50  0001 C CNN "SPURL"
 	1    5250 3900
 	1    0    0    -1
@@
 F 2 "Diodes_ThroughHole_jl:Diode_TO_220AC_Horizonal" H 4350 4050 50  0001 C CNN
 F 3 "http://www.vishay.com/docs/96244/vs-20etsm3_vs-20atsm3.pdf" H 4350 4050 50  0001 C CNN
+F 4 "-" H 0   0   50  0001 C CNN "MFR"
+F 5 "-" H 0   0   50  0001 C CNN "MPN"
+F 6 "-" H 0   0   50  0001 C CNN "SPR"
+F 7 "-" H 0   0   50  0001 C CNN "SPN"
+F 8 "-" H 0   0   50  0001 C CNN "SPURL"
 	1    4350 4050
 	0    1    1    0
 $EndComp
-Wire Wire Line
-	2750 3900 3100 3900
-Wire Wire Line
-	3400 3900 4350 3900
-Wire Wire Line
-	4350 3900 5100 3900
-Connection ~ 4350 3900
-Wire Wire Line
-	4350 3900 4350 2900
-Wire Wire Line
-	5400 3900 6000 3900
 $Comp
 L power:GNDPWR #PWR0501
@@
 	1    0    0    -1
 $EndComp
+Text Notes 6700 3750 2    50   ~ 0
+Solar 585V 8A Max
+Text HLabel 2750 3900 0    50   Input ~ 0
+Vbattery_in
+Text HLabel 6000 3900 2    50   Input ~ 0
+Vsolar_in
+Text HLabel 4350 2900 1    50   Output ~ 0
+Vout
+Text Notes 2250 3750 0    50   ~ 0
+Battery Boost 160V 6.25A
+Wire Wire Line
+	2750 3900 3100 3900
+Wire Wire Line
+	3400 3900 4350 3900
+Wire Wire Line
+	4350 3900 5100 3900
+Wire Wire Line
+	4350 3900 4350 2900
+Wire Wire Line
+	5400 3900 6000 3900
 Wire Wire Line
 	4350 4400 4350 4200
-Text Notes 2250 3750 0    50   ~ 0
-Battery Boost 160V 6.25A
+Connection ~ 4350 3900
 $EndSCHEMATC

Commit message: Finished adding digi key part numbers, for now git add *
Parts:
- D501, D502, D503: MFR - -> Vishay Semiconductor Diodes Division; MPN - -> VS-20ETS12-M3; SPN - -> VS-20ETS12-M3-ND; SPR - -> digikey
Changed lines of the file:
@@
 F 2 "Diodes_ThroughHole_jl:Diode_TO_220AC_Horizonal" H 3250 3900 50 0001 C CNN
 F 3 "http://www.vishay.com/docs/96244/vs-20etsm3_vs-20atsm3.pdf" H 3250 3900 50 0001 C CNN
-F 4 "-" H 0 0 50 0001 C CNN "MFR"
-F 5 "-" H 0 0 50 0001 C CNN "MPN"
-F 6 "-" H 0 0 50 0001 C CNN "SPR"
-F 7 "-" H 0 0 50 0001 C CNN "SPN"
+F 4 "Vishay Semiconductor Diodes Division" H 0 0 50 0001 C CNN "MFR"
+F 5 "VS-20ETS12-M3" H 0 0 50 0001 C CNN "MPN"
+F 6 "digikey" H 0 0 50 0001 C CNN "SPR"
+F 7 "VS-20ETS12-M3-ND" H 0 0 50 0001 C CNN "SPN"
 F 8 "-" H 0 0 50 0001 C CNN "SPURL"
 	1    3250 3900
@@
 F 2 "Diodes_ThroughHole_jl:Diode_TO_220AC_Horizonal" H 5250 3900 50 0001 C CNN
 F 3 "http://www.vishay.com/docs/96244/vs-20etsm3_vs-20atsm3.pdf" H 5250 3900 50 0001 C CNN
-F 4 "-" H 0 0 50 0001 C CNN "MFR"
-F 5 "-" H 0 0 50 0001 C CNN "MPN"
-F 6 "-" H 0 0 50 0001 C CNN "SPR"
-F 7 "-" H 0 0 50 0001 C CNN "SPN"
+F 4 "Vishay Semiconductor Diodes Division" H 0 0 50 0001 C CNN "MFR"
+F 5 "VS-20ETS12-M3" H 0 0 50 0001 C CNN "MPN"
+F 6 "digikey" H 0 0 50 0001 C CNN "SPR"
+F 7 "VS-20ETS12-M3-ND" H 0 0 50 0001 C CNN "SPN"
 F 8 "-" H 0 0 50 0001 C CNN "SPURL"
 	1    5250 3900
@@
 F 2 "Diodes_ThroughHole_jl:Diode_TO_220AC_Horizonal" H 4350 4050 50 0001 C CNN
 F 3 "http://www.vishay.com/docs/96244/vs-20etsm3_vs-20atsm3.pdf" H 4350 4050 50 0001 C CNN
-F 4 "-" H 0 0 50 0001 C CNN "MFR"
-F 5 "-" H 0 0 50 0001 C CNN "MPN"
-F 6 "-" H 0 0 50 0001 C CNN "SPR"
-F 7 "-" H 0 0 50 0001 C CNN "SPN"
+F 4 "Vishay Semiconductor Diodes Division" H 0 0 50 0001 C CNN "MFR"
+F 5 "VS-20ETS12-M3" H 0 0 50 0001 C CNN "MPN"
+F 6 "digikey" H 0 0 50 0001 C CNN "SPR"
+F 7 "VS-20ETS12-M3-ND" H 0 0 50 0001 C CNN "SPN"
 F 8 "-" H 0 0 50 0001 C CNN "SPURL"
 	1    4350 4050
