File: SolarDCSwitch.sch (KiCad schematic (older format))
At the start: 11 parts

Commit message: Added extra FET in Current sense Auto Ranging circuit to stop the conduction of the body diode of the single FET on the negative half of the mains cycle.  Also change the Values of all the TestPoints from TestPoint to a useful name either the voltage they should read or what they measure, also chaged there layer to front Silks so they can be used.
Parts:
- TP501: value TestPoint -> TP_Solar_Voltage
Changed lines of the file:
@@
 AR Path="/5F4EB1AC/5F487196" Ref="TP501"  Part="1"
 F 0 "TP501" H 4658 5968 50  0000 L CNN
-F 1 "TestPoint" H 4658 5877 50  0000 L CNN
+F 1 "TP_Solar_Voltage" H 4658 5877 50  0000 L CNN
 F 2 "TestPoint:TestPoint_Pad_3.0x3.0mm" H 4800 5850 50  0001 C CNN
 F 3 "~" H 4800 5850 50  0001 C CNN
