File: _autosave-GridTiedBatteryBoostConverter.kicad_pcb (KiCad board)
At the start: 2 copper layers, 270.1 x 143.1 mm, 116 parts, among them J101 Battery Connection, J103 Solar Panels, J401 Screw_Terminal_01x02, J402 AudioJack2_SwitchT, Q101 IXFP36N20X3, Q102 BC847B-13-F, Q103 SSM3K329R, Q104 SSM3J334R, Q201 SSM3K329R, Q202 SSM3K329R, Q203 SSM3J334R, Q301 BC847B-13-F, Q302 BC856B-13-F, Q305 TK32A12N1,S4X, Q306 TK32A12N1,S4X, SW201 SW_Push, SW202 SW_Push, SW203 SW_Push, U101 OPA2837DGK, U102 UCC2800DTR, U201 LCD 2004A, U202 Teensy-LC, U203 wizfi360, U301 FDA217, U302 LTC7138EMSE-PBF, U303 TPS560200, U304 TLV70430_SOT23-5

Commit message: Improved clearance of Vin into U302 as good as the package will allow. Also reduced clearance around the Teesy to 0.5mm, because I notice one for the grounds was not connected.
Parts:
- removed R403: 1K ohms .1%, Resistors_SMD:R_0805_HandSoldering
- added C201: 1uF X7R 25V 10%, Capacitors_SMD:C_0805_HandSoldering, F.Cu at (142.8, 129.9)
- added C202: 0.1uF X7R 25V 10%, Capacitors_SMD:C_0805_HandSoldering, F.Cu at (142.8, 128.0)
- added C203: 0.1uF X7R 25V 10%, Capacitors_SMD:C_0805_HandSoldering, F.Cu at (32.8, 127.8)
- added C204: 10uF X7R 25V 10%, Capacitors_SMD:C_1206_HandSoldering, F.Cu at (38.6, 124.8)
- added C205: 0.1uF X7R 25V 10%, Capacitors_SMD:C_0805_HandSoldering, F.Cu at (67.2, 129.2)
- added C301: 10uF X7R 25V 10%, Capacitors_SMD:C_1206_HandSoldering, F.Cu at (37.2, 108.1)
- added C302: 0.47uF X7R 25V 10%, Capacitors_SMD:C_0805_HandSoldering, F.Cu at (166.6, 96.9)
- added C304: 0.1uF X7R 25V 10%, Capacitors_SMD:C_0805_HandSoldering, F.Cu at (34.6, 108.8)
- added C305: 10uF X7R 25V 10%, Capacitors_SMD:C_1206_HandSoldering, F.Cu at (23.1, 111.8)
- added C307: 10uF X7R 25V 10%, Capacitors_SMD:C_1206_HandSoldering, F.Cu at (20.5, 111.8)
- added C315: 33uF X7R 16V 20%, Capacitors_SMD:C_1812_HandSoldering, F.Cu at (126.4, 77.8)
- added J202: Conn_01x03_Female, Pin_Headers:Pin_Header_Straight_1x03_Pitch2.54mm, F.Cu at (74.5, 133.8)
- added J203: I2C_BUS, Pin_Headers:Pin_Header_Straight_1x04_Pitch2.54mm, F.Cu at (153.3, 101.0)
- added JP201: SDA_EN, Pin_Headers:Pin_Header_Straight_1x02_Pitch2.54mm, F.Cu at (29.8, 137.6)
- added JP202: SCL_EN, Pin_Headers:Pin_Header_Straight_1x02_Pitch2.54mm, F.Cu at (29.8, 133.5)
- added JP203: BOOT_OPTION, Pin_Headers:Pin_Header_Straight_1x02_Pitch2.54mm, F.Cu at (38.1, 138.7)
- added L303: 15uH 730mA Sat, Inductors_jl:Inductor_1210_HandSoldering, F.Cu at (27.7, 112.5)
- added R208: 4K7 1%, Resistors_SMD:R_0805_HandSoldering, F.Cu at (139.9, 125.8)
- added R209: 15K 1%, Resistors_SMD:R_0805_HandSoldering, F.Cu at (40.2, 132.2)
- added R210: 15K 1%, Resistors_SMD:R_0805_HandSoldering, F.Cu at (34.1, 122.5)
- added R211: 4K7 1%, Resistors_SMD:R_0805_HandSoldering, F.Cu at (160.9, 95.6)
- added R212: 4K7 1%, Resistors_SMD:R_0805_HandSoldering, F.Cu at (157.3, 95.6)
- added R213: 15K 1%, Resistors_SMD:R_0805_HandSoldering, F.Cu at (66.0, 123.3)
- added R303: 61.9K 0.1%, Resistors_SMD:R_0805_HandSoldering, F.Cu at (21.8, 107.1)
- added R304: 20K 0.1%, Resistors_SMD:R_0805_HandSoldering, F.Cu at (26.4, 108.5)
- added REF**: MountingHole_3.2mm_M3_Pad, Mounting_Holes:MountingHole_3.2mm_M3_Pad, F.Cu at (141.8, 91.8)
- added REF**: MountingHole_3.2mm_M3_Pad, Mounting_Holes:MountingHole_3.2mm_M3_Pad, F.Cu at (278.1, 19.5)
- added REF**: MountingHole_3.2mm_M3_Pad, Mounting_Holes:MountingHole_3.2mm_M3_Pad, F.Cu at (278.1, 152.6)
- added REF**: MountingHole_3.2mm_M3_Pad, Mounting_Holes:MountingHole_3.2mm_M3_Pad, F.Cu at (18.0, 19.5)
- added REF**: MountingHole_3.2mm_M3_Pad, Mounting_Holes:MountingHole_3.2mm_M3_Pad, F.Cu at (18.0, 152.5)
- added TP101: TestPoint, Measurement_Points:Measurement_Point_Square-SMD-Pad_Big, F.Cu at (194.7, 102.7)
- added TP102: TestPoint, Measurement_Points:Measurement_Point_Square-SMD-Pad_Big, F.Cu at (194.8, 72.5)
- added TP103: TestPoint, Measurement_Points:Measurement_Point_Square-SMD-Pad_Big, F.Cu at (184.6, 98.2)
- added TP201: TestPoint, Measurement_Points:Measurement_Point_Square-SMD-Pad_Big, F.Cu at (118.3, 128.2)
- added TP202: TestPoint, Measurement_Points:Measurement_Point_Square-SMD-Pad_Big, F.Cu at (153.9, 126.0)
- added TP203: TestPoint, Measurement_Points:Measurement_Point_Square-SMD-Pad_Big, F.Cu at (171.8, 100.7)
- added TP301: TestPoint, Measurement_Points:Measurement_Point_Square-SMD-Pad_Big, F.Cu at (29.4, 103.0)
- added TP302: TestPoint, Measurement_Points:Measurement_Point_Square-SMD-Pad_Big, F.Cu at (26.1, 116.2)
- added TP303: TestPoint, Measurement_Points:Measurement_Point_Square-SMD-Pad_Big, F.Cu at (108.7, 91.3)
- added TP304: TestPoint, Measurement_Points:Measurement_Point_Square-SMD-Pad_Big, F.Cu at (148.3, 68.7)
- added TP305: TestPoint, Measurement_Points:Measurement_Point_Square-SMD-Pad_Big, F.Cu at (185.1, 124.9)
- added TP306: TestPoint, Measurement_Points:Measurement_Point_Square-SMD-Pad_Big, F.Cu at (94.5, 82.0)
- added TP307: TestPoint, Measurement_Points:Measurement_Point_Square-SMD-Pad_Big, F.Cu at (167.8, 87.2)
- added U204: ESP-WROOM-02U, RF_Module_jl:MODULE_ESP-WROOM-02U, F.Cu at (52.8, 130.7)
- added U305: REF2925AIDBZT, Package_TO_SOT_SMD:SOT-23_Handsoldering, F.Cu at (166.3, 101.0)
- added U306: TPS560200DBVR, Package_TO_SOT_SMD:SOT-23-5_HandSoldering, F.Cu at (31.1, 109.0)
- C101: value 220uF 200V 905 mOhm -> 220uF ALUM 200V 905 mOhm 20%
- C102: value 15uF 250VDC 3.9mOhm -> 15uF PP 250VDC 3.9mOhm
- C103: value 470uF 400V 130mOhm -> 470uF ALUM 400V 130mOhm 20%
- C104: value 70uF 500V 2.1mOhm PP film -> 70uF PP Film 500V 2.1mOhm
- C105: value 100 pF -> 100pF
- C106, C111, C115: value 1uF 25V X7R -> 1uF X7R 25V 10%
- C107, C112: value 0.1uF mlcc -> 0.1uF X7R 25V 10%
- C108: value 1uF 16V X7R -> 1uF X7R 25V 10%
- C109: value C 0.1uF mlcc -> 0.1uF X7R 25V 10%
- C110: value 6 pF -> 6pF C0G
- C113: value 1 nF -> 1nF
- C114: value 1 uF -> 1uF X7R 25V 10%
- C303: value 1uF 250V x7r -> 1uF X7R 250V 10%
- C306: value 33uF X7R 16V -> 33uF X7R 16V 20%
- C308: value 10uF 16V X7R -> 10uF X7R 25V 10%
- C309: value 0.1uF 16V X7R -> 0.1uF X7R 25V 10%
- C310, C311: value 10uF X7R 16V -> 10uF X7R 25V 10%
- C312: value 0.1 uF 16V X7R -> 0.1uF X7R 25V 10%
- C313: value 1 uF 25V X7R -> 1uF X7R 25V 10%
- C314: value 1uF 250V X7R -> 1uF X7R 250V 10%
- C401: value C_Small -> 1uF X7R 25V 10%
- Cint101: value 0.56uF 10% 16V mlcc -> 0.56uF X7R 16V 10%
- Crolloff101: value 68 pF 5% C0G mlcc -> 68pF C0G 5%
- Ct101: value 200pF 2% C0G mlcc -> 200pF C0G 2%
- D101: value 8A 200V 0.950V fwd -> 8A 200V 0.950V
- D102, D103, D401, D402: value BAV54S -> BAT54S; footprint Package_TO_SOT_SMD:SOT-23 -> Package_TO_SOT_SMD:SOT-23_Handsoldering
- F101: value fuse 25A 100V DC -> Fuse Holder
- L101: value 47uH 31A Sat 6.38m Ohm -> 47uH 31A Sat 6.38m Ohm
- L302: value 15uH 600mA Sat -> 15uH 730mA Sat
- Q101: footprint Transistors_ThroughHole_jl:TO-220 -> Transistors_ThroughHole_jl:TO-220_Horizontal_Offset_Drain
- Q305, Q306: value TK32A12N1,S4X -> IRFP4321PBF; footprint Transistors_ThroughHole_jl:TO-220 -> Transistors_ThroughHole_jl:TO-247-3_Horizontal_TabDown
- R101: value 0 Ohms -> 0R Ohms
- R102: value 82k 0.1% .25W -> 82K 0.1%
- R103: value 75k 0.1% 0.25W -> 75K 0.1%
- R104: value 1.5k 0.1% 0.25W -> 1.5K 0.1%
- R105: value 1k 0.1% 0.25W -> 1K 0.1%
- R106, R108: value 1k 1% -> 1K 1%
- R110: value 10 k 0.1% -> 10K 0.1%
- R111: value 330 Ohm .1% -> 330R 0.1%
- R112: value 330 Ohm 0.1% -> 330R 0.1%
- R113: value 10 ohm -> 10R 1%
- R114: value 2 mOhm 0.5W -> 2 mOhm Thick Film 1% 1W; footprint Resistors_SMD:R_0805_HandSoldering -> Resistors_SMD:R_1210_HandSoldering
- R115: value 1M Ohm 1% -> 1M 1%
- R116, R117: value 10k 0.1% -> 10K 0.1%
- R118, R119: value 330 Ohms 0.1% -> 330R 0.1%
- R120: value 2 mOhm 0.1% -> 2 mOhm Thick Film 1% 1W; footprint Resistors_SMD:R_0805_HandSoldering -> Resistors_SMD:R_1210_HandSoldering
- R201, R202, R203, R204: value 1K -> 1K 1%
- R205: value 100K Ohm -> 100K 1%
- R206: value 100 Ohm 1% -> 100R 1%
- R302: value 330 1% -> 330R 1%
- R309: value 196k 0.1% -> 196K 0.1%
- R311: value 20k 0.1% -> 20K 0.1%
- R401: value 10K ohms .1% -> 5.9K 0 .1%
- R402: value 1K ohms .1% -> 1K 0.1%
- R404: value 47 Ohms 0.1% -> 41.2 0.1%
- R405, R406: value 10K ohms 0.1% -> 10K 0.1%
- Rint1: value 1.0k Ohm .1% -> 1K 0.1%
- Rint2: value 1.5 k Ohm -> 1.5K 0.1%
- SW201: value SW_Push -> SW_Up
- SW202: value SW_Push -> SW_Down
- SW203: value SW_Push -> SW_Enter
- U101: value OPA2837DGK -> OPA2837IDGKR
- U201: value LCD 2004A -> LCD 2004A Right Angle Header 16 pin 2.54mm
- U203: value wizfi360 -> PCF8574ADWR; footprint WIZnet:wiznet360-pa -> Housings_SOIC:SOIC-16W_7.5x10.3mm_Pitch1.27mm
- U303: value TPS560200 -> TPS560200DBVR
- U304: value TLV70430_SOT23-5 -> TLV70430DBVT; footprint Package_TO_SOT_SMD:SOT-23-5 -> Package_TO_SOT_SMD:SOT-23-5_HandSoldering
- moved SW203 156.4 mm to (194.1, 154.8)
- moved SW201 125.3 mm to (52.5, 154.7)
- moved U203 112.2 mm to (133.8, 134.4), turned to 0 degrees
- moved R312 59.0 mm to (88.3, 90.3), turned to 180 degrees
- moved R301 57.2 mm to (88.3, 87.0), turned to 180 degrees
- moved R302 55.1 mm to (88.3, 82.0), turned to 180 degrees
- moved U301 45.8 mm to (80.1, 85.8), turned to 90 degrees
- moved C314 44.5 mm to (72.8, 94.7), turned to 0 degrees
- moved U202 39.5 mm to (165.6, 113.6), turned to 0 degrees
- moved Q302 37.9 mm to (77.2, 75.0), turned to 90 degrees
- moved D401 34.7 mm to (186.6, 117.5)
- moved Q203 32.1 mm to (156.2, 141.6), turned to 0 degrees
- moved R205 31.4 mm to (152.4, 141.4), turned to 270 degrees
- moved Q301 30.4 mm to (72.0, 75.0), turned to 90 degrees
- moved D402 26.6 mm to (193.4, 114.7)
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Connections:
- net /Sheet5F4EB1AB/Vout renamed /Vout
- net /Sheet5F4EB1AB/Vsolar_in renamed /Vsolar_in
- net Net-(C314-Pad2) renamed /PowerSupplies/Charger_FETs_Source
- net Net-(J401-Pad1) renamed /MainsPowerMonitor/AC_Mains_Phase
- net Net-(J401-Pad2) renamed /MainsPowerMonitor/AC_Mains_Neutral
- net Net-(Q101-Pad1) renamed /GateDrive
- net Net-(Q301-Pad2) renamed /PowerSupplies/Charger_Fets_GateDrive
- C104 pad 3: Net-(C104-Pad3) -> 0
- J103 pad 2: 0 -> Net-(J103-Pad2)
- J103 pad 3: 0 -> Net-(J103-Pad2)
- J402 pad RN: Net-(C401-Pad1) -> (no net)
- J402 pad TN: Net-(C401-Pad1) -> (no net)
- R118 pad 2: 0 -> Net-(J103-Pad2)
- R119 pad 2: Net-(C104-Pad3) -> 0
- R120 pad 1: 0 -> Net-(J103-Pad2)
- R120 pad 2: Net-(C104-Pad3) -> 0
- R402 pad 2: Net-(R402-Pad2) -> Net-(C401-Pad1)
- R405 pad 1: +3.3V_TEENSY_OUT -> /+2.5V_REF
- TR401 pad 5: Net-(C401-Pad1) -> Net-(R401-Pad1)
- TR401 pad 6: Net-(R401-Pad1) -> Net-(C401-Pad1)
- TR401 pad 7: Net-(C401-Pad1) -> Net-(R401-Pad1)
- TR401 pad 8: Net-(R401-Pad1) -> Net-(C401-Pad1)
- U202 pad 12: Net-(U202-Pad12) -> Net-(SW201-Pad2)
- U202 pad 2: Net-(U202-Pad2) -> /Teensy-LC/mcu_wifi_rx
- U202 pad 23: LCD_ON_OFF -> Mains_Voltage
- U202 pad 24: /Teensy-LC/LCD_DB7 -> Mains_Current
- U202 pad 25: /Teensy-LC/LCD_DB6 -> Net-(U202-Pad25)
- U202 pad 26: /Teensy-LC/LCD_DB5 -> Net-(U202-Pad26)
- U202 pad 27: /Teensy-LC/LCD_EN -> /Teensy-LC/BOOST_ON_OFF
- U202 pad 28: /Teensy-LC/LCD_RW -> Net-(U202-Pad28)
- U202 pad 29: Net-(U202-Pad29) -> SCL1
- U202 pad 3: Net-(U202-Pad3) -> /Teensy-LC/mcu_wifi_tx
- U202 pad 30: Net-(SW201-Pad2) -> SDA1
- U202 pad 35: Net-(U202-Pad35) -> /+2.5V_REF
- U202 pad 36: Mains_Current -> Net-(U202-Pad36)
- U202 pad 37: Mains_Voltage -> Net-(U202-Pad37)
- U202 pad 5: Net-(U202-Pad5) -> /Teensy-LC/wifi_en
- U202 pad 6: /Teensy-LC/LCD_RS -> Net-(U202-Pad6)
- U202 pad 7: /Teensy-LC/BOOST_ON_OFF -> Net-(U202-Pad7)
- U202 pad 8: /Teensy-LC/LCD_DB4 -> Net-(U202-Pad8)
- U203 pad 1: Net-(U203-Pad1) -> 0
- U203 pad 10: Net-(U203-Pad10) -> /Teensy-LC/LCD_RW
- U203 pad 11: Net-(U203-Pad11) -> /Teensy-LC/LCD_RS
- U203 pad 12: Net-(U203-Pad12) -> LCD_ON_OFF
- U203 pad 14: Net-(U203-Pad14) -> SCL1
- U203 pad 15: Net-(U203-Pad15) -> SDA1
- U203 pad 16: Net-(U203-Pad16) -> +3.3V_TEENSY_OUT
- U203 pad 2: Net-(U203-Pad2) -> 0
- U203 pad 3: Net-(U203-Pad3) -> 0
- U203 pad 4: Net-(U203-Pad4) -> /Teensy-LC/LCD_DB4
- U203 pad 5: Net-(U203-Pad5) -> /Teensy-LC/LCD_DB5
- U203 pad 6: Net-(U203-Pad6) -> /Teensy-LC/LCD_DB6
- U203 pad 7: Net-(U203-Pad7) -> /Teensy-LC/LCD_DB7
- U203 pad 8: Net-(U203-Pad8) -> 0
- U203 pad 9: Net-(U203-Pad9) -> /Teensy-LC/LCD_EN
Routing:
- net SDA1: track 0.00 -> 215.3 mm, vias 0 -> 4
- net SCL1: track 0.00 -> 211.8 mm, vias 0 -> 6
- net Net-(SW203-Pad1): track 189.9 -> 37.6 mm, vias 6 -> 0
- net /Teensy-LC/wifi_en: track 0.00 -> 145.5 mm, vias 0 -> 2
- net Net-(J103-Pad2): track 0.00 -> 135.4 mm, vias 0 -> 3
- net Net-(SW201-Pad2): track 16.0 -> 147.4 mm
- net 0: track 214.5 -> 335.6 mm, vias 59 -> 88
- net +11V: track 60.3 -> 178.4 mm
- net /Teensy-LC/mcu_wifi_tx: track 0.00 -> 100.1 mm
- net /Teensy-LC/mcu_wifi_rx: track 0.00 -> 99.5 mm
- net /+2.5V_REF: track 0.00 -> 98.0 mm, vias 0 -> 2
- net Net-(C104-Pad3): track 94.2 -> 0.00 mm
- net +5V: track 333.4 -> 420.4 mm
- net +3.3V_wifi_only: track 0.00 -> 74.3 mm
- net Mains_Current: track 72.4 -> 141.1 mm, vias 2 -> 0
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Other:
- outline, holes or cut-outs redrawn
- net class AC_Mains added: clearance 2.5, trace_width 1, via_dia 1.2, via_drill 0.6
- net class ChargerConnection added: clearance 1.1, trace_width 8, via_dia 5, via_drill 2.5
- net class ChargerFetsGateDrive added: clearance 1.1, trace_width 1, via_dia 1.2, via_drill 0.6
- board text added: "+ Bat -"
- board text added: "+ Solar Panels -"
- board text added: "- Charger +"
- board text added: "- Inverter +"
- board text added: "Gnd"
- board text added: "I2C_BUS 3.3V GND SDA1 SCL"
- board text added: "Rx"
- board text added: "Tx"
- board text added: "Voltage Sense Phase Neutral"
- board text removed: "Inverter"
