File: Teensy-LC.sch (KiCad schematic (older format))
At the start: 37 parts, among them J202 Conn_01x03_Female, J203 I2C_BUS, Q201 SSM3K329R, Q202 SSM3K329R, Q203 SSM3J334R, SW201 SW_Up, SW202 SW_Down, SW203 SW_Enter, U201 LCD 2004A Right Angle Header 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, U202 Teensy-LC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

Commit message: Added extra FET in Current sense Auto Ranging circuit to stop the conduction of the body diode of the single FET on the negative half of the mains cycle.  Also change the Values of all the TestPoints from TestPoint to a useful name either the voltage they should read or what they measure, also chaged there layer to front Silks so they can be used.
Parts:
- TP201: value TestPoint -> TP_LCD_On
- TP202: value TestPoint -> TP +3.3V
- TP203: value TestPoint -> TP_Boost_On
Changed lines of the file:
@@
 AR Path="/5EF73D52/604D2532" Ref="TP201"  Part="1"
 F 0 "TP201" H 1208 4518 50  0000 L CNN
-F 1 "TestPoint" H 1208 4427 50  0000 L CNN
+F 1 "TP_LCD_On" H 1208 4427 50  0000 L CNN
 F 2 "TestPoint:TestPoint_Pad_3.0x3.0mm" H 1350 4400 50  0001 C CNN
 F 3 "~" H 1350 4400 50  0001 C CNN
@@
 AR Path="/5EF73D52/604DC721" Ref="TP202"  Part="1"
 F 0 "TP202" H 7758 4568 50  0000 L CNN
-F 1 "TestPoint" H 7758 4477 50  0000 L CNN
+F 1 "TP +3.3V" H 7758 4477 50  0000 L CNN
 F 2 "TestPoint:TestPoint_Pad_3.0x3.0mm" H 7900 4450 50  0001 C CNN
 F 3 "~" H 7900 4450 50  0001 C CNN
@@
 AR Path="/5EF73D52/604F5CFE" Ref="TP203"  Part="1"
 F 0 "TP203" H 9258 5618 50  0000 L CNN
-F 1 "TestPoint" H 9258 5527 50  0000 L CNN
+F 1 "TP_Boost_On" H 9258 5527 50  0000 L CNN
 F 2 "TestPoint:TestPoint_Pad_3.0x3.0mm" H 9400 5500 50  0001 C CNN
 F 3 "~" H 9400 5500 50  0001 C CNN
